File: kicad/pioneer.kicad_pcb (KiCad board)
At the start: 2 copper layers, 85.3 x 54.3 mm, 13 parts, among them SW1 SW_Push, SW2 SW_Push, SW3 SW_Push, SW4 SW_Push, U1 XIAO-RP2040-DIP

Commit message: Updated project KiCad files
Routing:
- net GND: track 223.9 -> 229.8 mm, vias 0 -> 1
- net LED3: track 58.0 -> 60.5 mm
